Commit message: feat: add front right axle with visual and collision properties in URDF

File: Resources/robots/pioneer.urdf (robot description, URDF)
Before this commit: robot pioneer3at_body, 6 links, 5 joints
Links:
- added link p3at_front_right_axle, mass 0.1; collision box size=0.01 0.01 0.01; visual mesh filename=/home/tashi/Desktop/project-mobrob/Resources/meshes/p3at_me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
Joints:
- added joint base_front_right_axle_joint: type fixed, parent base_link, child p3at_front_right_axle, origin xyz=0.135 -0.156 0.111 rpy=0 0 0

Commit message: feat: add front right hub with visual and collision properties in URDF

File: Resources/robots/pioneer.urdf (robot description, URDF)
Before this commit: robot pioneer3at_body, 7 links, 6 joints
Links:
- added link p3at_front_right_hub, mass 0.1; collision box size=0.01 0.01 0.01; visual mesh filename=/home/tashi/Desktop/project-mobrob/Resources/meshes/p3at_me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
Joints:
- added joint base_front_right_hub_joint: type fixed, parent p3at_front_right_axle, child p3at_front_right_hub, origin xyz=0 -0.041 0 rpy=0 0 0

Commit message: feat: add front right wheel, complete

File: Resources/robots/pioneer.urdf (robot description, URDF)
Before this commit: robot pioneer3at_body, 8 links, 7 joints
Links:
- added link p3at_front_right_wheel, mass 0.5; collision mesh filename=/home/tashi/Desktop/project-mobrob/Resources/meshes/p3at_me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; visual mesh filename=/home/tashi/Desktop/project-mobrob/Resources/meshes/p3at_me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
Joints:
- added joint p3at_front_right_wheel_joint: type continuous, parent p3at_front_right_hub, child p3at_front_right_wheel, origin xyz=0 0 0 rpy=0 0 0, axis 0 1 0, limit effort=100 velocity=100

Commit message: feat: add back left axle

File: Resources/robots/pioneer.urdf (robot description, URDF)
Before this commit: robot pioneer3at_body, 9 links, 8 joints
Links:
- added link p3at_back_left_axle, mass 0.1; collision box size=0.01 0.01 0.01; visual mesh filename=/home/tashi/Desktop/project-mobrob/Resources/meshes/p3at_me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
Joints:
- added joint base_back_left_axle_joint: type fixed, parent base_link, child p3at_back_left_axle, origin xyz=-0.135 0.156 0.111 rpy=0 0 0

Commit message: feat: add back left hub

File: Resources/robots/pioneer.urdf (robot description, URDF)
Before this commit: robot pioneer3at_body, 10 links, 9 joints
Links:
- added link p3at_back_left_hub, mass 0.1; collision box size=0.01 0.01 0.01; visual mesh filename=/home/tashi/Desktop/project-mobrob/Resources/meshes/p3at_me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
Joints:
- added joint base_back_left_hub_joint: type fixed, parent p3at_back_left_axle, child p3at_back_left_hub, origin xyz=0 0.041 0 rpy=0 0 0

Commit message: feat: add back left wheel with visual and collision properties in URDF, complete

File: Resources/robots/pioneer.urdf (robot description, URDF)
Before this commit: robot pioneer3at_body, 11 links, 10 joints
Links:
- added link p3at_back_left_wheel, mass 0.5; collision mesh filename=/home/tashi/Desktop/project-mobrob/Resources/meshes/p3at_me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; visual mesh filename=/home/tashi/Desktop/project-mobrob/Resources/meshes/p3at_me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
Joints:
- added joint p3at_back_left_wheel_joint: type continuous, parent p3at_back_left_hub, child p3at_back_left_wheel, origin xyz=0 0 0 rpy=0 0 0, axis 0 1 0, limit effort=100 velocity=100

Commit message: feat: add back right axle

File: Resources/robots/pioneer.urdf (robot description, URDF)
Before this commit: robot pioneer3at_body, 12 links, 11 joints
Links:
- added link p3at_back_right_axle, mass 0.1; collision box size=0.01 0.01 0.01; visual mesh filename=/home/tashi/Desktop/project-mobrob/Resources/meshes/p3at_me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
Joints:
- added joint base_back_right_axle_joint: type fixed, parent base_link, child p3at_back_right_axle, origin xyz=-0.135 -0.156 0.111 rpy=0 0 0

Commit message: feat: add back right hub

File: Resources/robots/pioneer.urdf (robot description, URDF)
Before this commit: robot pioneer3at_body, 13 links, 12 joints
Links:
- added link p3at_back_right_hub, mass 0.1; collision box size=0.01 0.01 0.01; visual mesh filename=/home/tashi/Desktop/project-mobrob/Resources/meshes/p3at_me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
Joints:
- added joint base_back_right_hub_joint: type fixed, parent p3at_back_right_axle, child p3at_back_right_hub, origin xyz=0 -0.041 0 rpy=0 0 0

Commit message: feat: add back right wheel with visual and collision properties in URDF, complete

File: Resources/robots/pioneer.urdf (robot description, URDF)
Before this commit: robot pioneer3at_body, 14 links, 13 joints
Links:
- added link p3at_back_right_wheel, mass 0.5; collision mesh filename=/home/tashi/Desktop/project-mobrob/Resources/meshes/p3at_me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; visual mesh filename=/home/tashi/Desktop/project-mobrob/Resources/meshes/p3at_me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
Joints:
- added joint p3at_back_right_wheel_joint: type continuous, parent p3at_back_right_hub, child p3at_back_right_wheel, origin xyz=0 0 0 rpy=0 0 0, axis 0 1 0, limit effort=100 velocity=100

Commit message: feat: add laser joint and frame with lidar sensor configuration in URDF

File: Resources/robots/pioneer.urdf (robot description, URDF)
Before this commit: robot pioneer3at_body, 15 links, 14 joints
Links:
- added link laser_frame, mass 1e-5; collision box size=0.01 0.01 0.01; visual mesh filename=/home/tashi/Desktop/project-mobrob/Resources/meshes/hokuyo1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
Joints:
- added joint laser_joint: type fixed, parent chassis, child laser_frame, origin xyz=0.2 0 0.104 rpy=0 0 0

Commit message: feat: add camera joint and frame with sensor configuration in URDF

File: Resources/robots/pioneer.urdf (robot description, URDF)
Before this commit: robot pioneer3at_body, 16 links, 15 joints
Links:
- added link cam_frame; visual box size=0.01 0.05 0.01
- added link cam_optical_link
Joints:
- added joint cam_joint: type fixed, parent chassis, child cam_frame, origin xyz=0.24 0 0.084 rpy=0 0 0
- added joint cam_optical_joint: type fixed, parent cam_frame, child cam_optical_link, origin xyz=0 0 0 rpy=-1.5708 0 -1.5708
